File: beginner_board.kicad_pcb (KiCad board)
At the start: 2 copper layers, 65 x 65 mm, 53 parts, among them J1 I2C_STANDARD, J10 ENCODER, J11 SERIAL, J13 SW_JUMPER, J14 SW2_JUMPER, J2 INPUT_VCC, J3 VOLTAGE_SELECTOR, J4 RELAY_OUTPUT, J5 STEPPER_OUTPUT, J7 MOTOR1, J8 MOTOR2, J9 STEPPER_POWER, K1 G5Q-1A, Q1 BC547, SW1 SW_Push, SW2 SW_Push, U1 L7805, U2 ULN2003, U3 L293D

Commit message: new design with smd
Parts:
- removed C6: CP, Capacitors_THT:CP_Radial_D6.3mm_P2.50mm
- removed D6: LED, LEDs:LED_D3.0mm
- removed D8: D, Diodes_THT:D_A-405_P2.54mm_Vertical_KathodeUp
- removed MK1: Mounting_Hole, Mounting_Holes:MountingHole_3.2mm_M3_Pad_Via
- removed R12: 10K, Resistors_SMD:R_0805
- removed R13, R15: 1K, Resistors_SMD:R_0805
- removed TP1, TP2: TEST, Aesthetics:FIDUCIAL-1X2
- added D4: D, Diodes_SMD:D_SMA, F.Cu at (143.9, 123.6)
- added G***: LOGO, logos:SENSA_13x6, F.Cu at (158.5, 89.4)
- added G***: LOGO, logos:SENSA_6x3, F.Cu at (134.4, 128.7)
- added G***: LOGO, logos:AISLER_3x2, F.Cu at (144.5, 128.7)
- added G***: LOGO, logos:AISLER_9x5, B.Cu at (147.3, 116.0)
- added G***: LOGO, logos:SENSA_15x6, B.Cu at (162.8, 116.2)
- added J6: Conn_01x02, Resistors_SMD:R_1206, F.Cu at (160.0, 120.5)
- C1, C4, C5: value CP -> 100u; footprint Capacitors_THT:CP_Radial_D6.3mm_P2.50mm -> Capacitors_Tantalum_SMD:CP_Tantalum_Case-B_EIA-3528-21_Hand
- C2, C3: value C -> 100n
- D1, D5: footprint Diodes_THT:D_A-405_P2.54mm_Vertical_KathodeUp -> Diodes_SMD:D_SMA
- Q1: value BC547 -> BC847; footprint TO_SOT_Packages_THT:TO-92_Molded_Narrow -> TO_SOT_Packages_SMD:SOT-23
- R6: value 2K2 -> 10K
- RV1: footprint Potentiometers:Potentiometer_WirePads -> Potentiometers:Potentiometer_WirePads_Small
- U2: footprint Housings_DIP:DIP-16_W7.62mm -> Housings_SOIC:SOIC-16_3.9x9.9mm_Pitch1.27mm
- U3: value L293D -> TB6612FNG; footprint Housings_DIP:DIP-16_W7.62mm -> Housings_SSOP:SSOP-24_5.3x8.2mm_Pitch0.65mm
- moved SW1 118.9 mm to (108.5, 80.7), turned to 90 degrees
- moved D1 100.2 mm to (137.9, 79.2), turned to 90 degrees
- moved J14 92.6 mm to (116.7, 88.4), turned to 270 degrees
- moved D2 91.5 mm to (168.2, 89.0), turned to 270 degrees
- moved J10 88.6 mm to (119.6, 89.5), turned to 180 degrees
- moved U1 87.0 mm to (146.1, 80.3), turned to 90 degrees
- moved J13 86.3 mm to (116.7, 85.6), turned to 270 degrees
- moved J1 85.6 mm to (149.2, 88.3), turned to 270 degrees
- moved K1 85.0 mm to (140.1, 117.9), turned to 180 degrees
- moved C2 83.2 mm to (141.2, 81.3), turned to 90 degrees
- moved J7 83.1 mm to (111.5, 103.0), turned to 90 degrees
- moved SW2 82.3 mm to (108.5, 89.2), turned to 270 degrees
- moved C3 81.6 mm to (149.6, 79.2), turned to 270 degrees
- moved U3 81.5 mm to (127.7, 102.9)
- moved R8 80.9 mm to (115.2, 90.9), turned to 180 degrees
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Connections:
- D3 pad 2: A1 -> +5V
- D5 pad 1: +5V -> STEPPER_PWR
- J9 pad 1: GND -> Net-(D5-Pad2)
- J9 pad 2: Net-(D8-Pad2) -> GND
- K1 pad 1: Net-(D5-Pad2) -> Net-(D4-Pad2)
- Q1 pad 1: Net-(D5-Pad2) -> Net-(Q1-Pad1)
- Q1 pad 2: Net-(Q1-Pad2) -> GND
- Q1 pad 3: GND -> Net-(D4-Pad2)
- R10 pad 1: Net-(Q1-Pad2) -> Net-(Q1-Pad1)
- R11 pad 2: A2 -> A1
- R2 pad 1: A0 -> A6
- R4 pad 2: A0 -> A6
- R6 pad 1: A2 -> A1
- U3 pad 1: +5V -> M_O_11
- U3 pad 10: D9 -> GND
- U3 pad 12: GND -> M_O_21
- U3 pad 13: GND -> +12V
- U3 pad 14: M_O_22 -> +12V
- U3 pad 16: MOTOR_PWR -> A0
- U3 pad 2: D5 -> M_O_11
- U3 pad 3: M_O_11 -> GND
- U3 pad 5: GND -> M_O_12
- U3 pad 7: D6 -> M_O_22
- U3 pad 8: +5V -> M_O_22
- U3 pad 9: +5V -> GND
Routing:
- net +5V: track 0.00 -> 194.8 mm, vias 0 -> 4
- net +12V: track 0.00 -> 170.0 mm
- net GND: track 0.00 -> 124.9 mm, vias 0 -> 24
- net D2: track 0.00 -> 62.3 mm
- net D3: track 0.00 -> 57.5 mm
- net A7: track 0.00 -> 43.4 mm
- net A0: track 0.00 -> 32.7 mm
- net D9: track 0.00 -> 30.9 mm, vias 0 -> 1
- net D10: track 0.00 -> 29.3 mm, vias 0 -> 1
- net A1: track 0.00 -> 27.9 mm, vias 0 -> 1
- net D4: track 0.00 -> 27.2 mm
- net A2: track 0.00 -> 26.5 mm, vias 0 -> 1
- net M_O_22: track 0.00 -> 25.9 mm
- net A3: track 0.00 -> 25.7 mm, vias 0 -> 1
- net D6: track 0.00 -> 24.9 mm, vias 0 -> 1
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- added copper zone on B.Cu, net GND
- added copper zone on F.Cu, net GND
- added copper zone on F.Cu, net STEPPER_PWR
Other:
- board size 65 x 65 mm -> 72 x 56 mm
- board text added: "+"
- board text added: "+ -"
- board text added: "-"
- board text added: "- +"
- board text added: "12V S 5V"
- board text added: "5V"
- board text added: "6V-15V"
- board text added: "7V-25V"
- board text added: "A/2"
- board text added: "A1 A2 B1 B2"
- board text added: "B/3"
- board text added: "BEGINNER BOARD V1.1 2018 OCTOBER"
- board text added: "Designed by S. Gal & A. Wasi"
- board text added: "G TX RX"
- board text added: "GND"
- board text added: "MADE BY"
- board text added: "MOTOR 1"
- board text added: "MOTOR 2"
- board text added: "POWER ON"
- board text added: "SCL"
- board text added: "SDA"
- board text added: "SW 1"
- board text added: "SW 2"
- board text added: "USB"
- board text added: "Use M3 -----> Screw"
- board text added: "Use M3 <--- Screw"
- board text added: "WITH"
