File: beginner_board.sch (KiCad schematic (older format))
At the start: 67 parts, among them J1 I2C_STANDARD, J10 Conn_01x04, J11 Conn_01x03, J12 Conn_01x02, J13 Conn_01x02, J14 Conn_01x02, J2 Screw_Terminal_01x02, J3 Conn_01x03, J4 Screw_Terminal_01x02, J5 Screw_Terminal_01x04, J6 Screw_Terminal_01x02, J7 Screw_Terminal_01x02, J8 Screw_Terminal_01x02, J9 Screw_Terminal_01x02, K1 G5Q-1A, Q1 BC547, Q2 BC547, Q3 BC547, SW1 SW_Push, SW2 SW_Push, U1 L7805, U2 L293D, U3 L293D

Commit message: DEV for download
Parts:
- removed D4: LED, LEDs:LED_D3.0mm, symbol LED
- removed D7: D, Diodes_THT:D_A-405_P2.54mm_Vertical_KathodeUp, symbol D
- removed J12: Conn_01x02, Pin_Headers:Pin_Header_Straight_1x02_Pitch2.54mm, symbol Conn_01x02
- removed J6: Screw_Terminal_01x02, TerminalBlocks_Phoenix:TerminalBlock_Phoenix_MKDS1.5-2pol, symbol Screw_Terminal_01x02
- removed Q2, Q3: BC547, TO_SOT_Packages_THT:TO-92_Molded_Narrow, symbol BC547
- removed R14: 10K, Resistors_THT:R_Box_L8.4mm_W2.5mm_P5.08mm, symbol R
- removed TP10, TP11, TP12, TP3, TP4, TP5, TP6, TP7, TP8, TP9: TEST, Aesthetics:FIDUCIAL-1X2, symbol TEST
- removed U2: L293D, Housings_DIP:DIP-16_W7.62mm, symbol L293D
- added C5, C6: CP, Capacitors_THT:CP_Radial_D6.3mm_P2.50mm, symbol CP
- added MK3: Mounting_Hole, Mounting_Holes:MountingHole_3.2mm_M3_Pad_Via, symbol Mounting_Hole
- added U2: ULN2003, Housings_DIP:DIP-16_W7.62mm, symbol ULN2003
- D2, D3: footprint LEDs:LED_D3.0mm -> LEDs:LED_0805
- J10: value Conn_01x04 -> ENCODER
- J11: value Conn_01x03 -> SERIAL
- J13: value Conn_01x02 -> SW_JUMPER
- J14: value Conn_01x02 -> SW2_JUMPER
- J2: value Screw_Terminal_01x02 -> INPUT_VCC
- J3: value Conn_01x03 -> VOLTAGE_SELECTOR
- J4: value Screw_Terminal_01x02 -> RELAY_OUTPUT
- J5: value Screw_Terminal_01x04 -> STEPPER_OUTPUT
- J7: value Screw_Terminal_01x02 -> MOTOR1
- J8: value Screw_Terminal_01x02 -> MOTOR2
- J9: value Screw_Terminal_01x02 -> STEPPER_POWER
- R1, R10, R11, R15, R2, R3, R4, R5, R7, R8, R9: footprint Resistors_THT:R_Box_L8.4mm_W2.5mm_P5.08mm -> Resistors_SMD:R_0805
- R12: value 1K -> 10K; footprint Resistors_THT:R_Box_L8.4mm_W2.5mm_P5.08mm -> Resistors_SMD:R_0805
- R13: value 10K -> 1K; footprint Resistors_THT:R_Box_L8.4mm_W2.5mm_P5.08mm -> Resistors_SMD:R_0805
- R6: value 1K -> 2K2; footprint Resistors_THT:R_Box_L8.4mm_W2.5mm_P5.08mm -> Resistors_SMD:R_0805
- RV1: footprint Potentiometers:Potentiometer_Alps_RK09K_Horizontal -> Potentiometers:Potentiometer_WirePads
- SW1, SW2: footprint Buttons_Switches_THT:SW_PUSH_6mm -> Buttons_Switches_SMD:SW_SPST_EVQPE1
Connections:
- net STP_CON1 is gone; now on net A6: R12.1
- net STP_CON2 is gone; now on net GND: R11.1
- net +5V: no longer R13.1
- net A1: now also D3.2 (A); no longer R1.2, RV1.2
- net A2: now also R11.2, R6.1
- net A3: now also D2.2 (A)
- net A6: now also R13.2
- net A7: now also R1.2, RV1.2
- net D11: now also U2.3 (I3)
- net D12: now also U2.4 (I4)
- net D4: now also U2.1 (I1); no longer D2.2 (A)
- net D8: now also U2.2 (I2); no longer D3.2 (A)
- net GND: now also R13.1, C5.2, C6.2, U2.8 (GND); no longer R6.1
- net MOTOR_PWR: now also R12.2, C6.1
- net STEPPER_PWR: now also R6.2, C5.1, U2.9 (COM)
- net at J5.4 (Pin_4): now also U2.13 (O4)
- net at J5.3 (Pin_3): now also U2.14 (O3)
- net at J5.1 (Pin_1): now also U2.16 (O1)
- net at J5.2 (Pin_2): now also U2.15 (O2)
- no-connect marks 4 -> 10
Other:
- note added: "ARDUINO SECTION"
- note added: "DEBUG SECTION"
- note added: "MOTOR SECTION"
- note added: "POWER SECTION"
- note added: "RELAY SECTION"
- note added: "STEPPER SECTION"
- note removed: "Arduino NANO V3 Pinout"
- note removed: "BUTTONS & ENCODER"
- note removed: "DUAL MOTOR setup with L293D"
- note removed: "I2C pinout\n"
- note removed: "LED"
- note removed: "MOUNT HOLES"
- note removed: "POT"
- note removed: "POWER"
- note removed: "RELAY"
- note removed: "STEPPER MODULE with L293D"
- moved on the sheet: A1, C1, C2, C3, C4, D1, D2, D3, D5, D6, D8, J1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

Commit message: new design with smd
Parts:
- removed C6: CP, Capacitors_THT:CP_Radial_D6.3mm_P2.50mm, symbol CP
- removed D6: LED, LEDs:LED_D3.0mm, symbol LED
- removed D8: D, Diodes_THT:D_A-405_P2.54mm_Vertical_KathodeUp, symbol D
- removed MK1: Mounting_Hole, Mounting_Holes:MountingHole_3.2mm_M3_Pad_Via, symbol Mounting_Hole
- removed Q1: BC547, TO_SOT_Packages_THT:TO-92_Molded_Narrow, symbol BC547
- removed R12: 10K, Resistors_SMD:R_0805, symbol R
- removed R13, R15: 1K, Resistors_SMD:R_0805, symbol R
- removed TP1, TP2: TEST, Aesthetics:FIDUCIAL-1X2, symbol TEST
- removed U3: L293D, Housings_DIP:DIP-16_W7.62mm, symbol L293D
- added D4: D, Diodes_SMD:D_SMA, symbol D
- added J6: Conn_01x02, Resistors_SMD:R_1206, symbol Conn_01x02
- added Q1: BC847, TO_SOT_Packages_SMD:SOT-23, symbol BC847
- added U3: TB6612FNG, Housings_SSOP:SSOP-24_5.3x8.2mm_Pitch0.65mm, symbol TB6612FNG
- C1, C4, C5: value CP -> 100u; footprint Capacitors_THT:CP_Radial_D6.3mm_P2.50mm -> Capacitors_Tantalum_SMD:CP_Tantalum_Case-B_EIA-3528-21_Hand
- C2, C3: value C -> 100n
- D1, D5: footprint Diodes_THT:D_A-405_P2.54mm_Vertical_KathodeUp -> Diodes_SMD:D_SMA
- R6: value 2K2 -> 10K
- RV1: footprint Potentiometers:Potentiometer_WirePads -> Potentiometers:Potentiometer_WirePads_Small
- U2: footprint Housings_DIP:DIP-16_W7.62mm -> Housings_SOIC:SOIC-16_3.9x9.9mm_Pitch1.27mm
Connections:
- net +12V: now also J6.1 (Pin_1), U3.13 (VM2), U3.14 (VM3), U3.24 (VM1)
- net +5V: now also D3.2 (A), D4.1 (K), U3.19 (STBY), U3.20 (VCC); no longer D5.1 (K)
- net A0: now also U3.16 (BIN2); no longer R2.1, R4.2
- net A1: now also R11.2, R6.1; no longer D3.2 (A)
- net A2: now also U3.17 (BIN1); no longer R11.2, R6.1
- net A6: now also R2.1, R4.2
- net D10: now also U3.15 (PWMB)
- net D5: now also U3.23 (PWMA)
- net D6: now also U3.22 (AIN2)
- net D9: now also U3.21 (AIN1)
- net GND: now also J9.2 (Pin_2), Q1.2 (E), U3.10 (PGND2), U3.18 (GND), U3.3 (PGND1), U3.4 (PGND1), U3.9 (PGND2); no longer J9.1 (Pin_1)
- net M_O_11: now also U3.1 (A01), U3.2 (A01)
- net M_O_12: now also U3.5 (A02), U3.6 (A02)
- net M_O_21: now also U3.11 (B01), U3.12 (B01)
- net M_O_22: now also U3.7 (B02), U3.8 (B02)
- net STEPPER_PWR: now also D5.1 (K), J6.2 (Pin_2)
- net at K1.1: now also D4.2 (A), Q1.3 (C); no longer D5.2 (A)
- net at R10.1: now also Q1.1 (B)
- new net: D5.2 (A), J9.1 (Pin_1)
Other:
- moved on the sheet: A1, D2, D3, J1, J11, J5, J7, J8, J9, MK4, R1, R3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
